Commit message: Fix the gripper collision mesh

File: source/assembly_benchmark/assembly_benchmark/assets/robots/r1_pro/robot.urdf (robot description, URDF)
Before this commit: robot r1_pro_with_gripper, 36 links, 35 joints
Links:
- link left_gripper_finger_link1: geometry collision mesh filename=meshes/left_gripper_finger_link1_collision.STL; visual mesh filename=meshes/left_gripper_finger_link1.obj
- link left_gripper_finger_link2: geometry collision mesh filename=meshes/left_gripper_finger_link2_collision.STL; visual mesh filename=meshes/left_gripper_finger_link2.obj
- link right_gripper_finger_link1: geometry collision mesh filename=meshes/right_gripper_finger_link1_collision.STL; visual mesh filename=meshes/right_gripper_finger_link1.obj
- link right_gripper_finger_link2: geometry collision mesh filename=meshes/right_gripper_finger_link2_collision.STL; visual mesh filename=meshes/right_gripper_finger_link2.obj
