Commit message: Added tactile sensors to the gripper.

File: source/assembly_benchmark/assembly_benchmark/assets/robots/r1_pro/robot.urdf (robot description, URDF)
Before this commit: robot r1_pro_with_gripper, 36 links, 35 joints
Links:
- added link left_gripper_tactile_pad1, mass 0.001; collision mesh filename=../../sensors/vt_refine_tactile/r1_pro_gripper_finger_link1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; visual mesh filename=../../sensors/vt_refine_tactile/r1_pro_gripper_finger_link1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
- added link left_gripper_tactile_pad2, mass 0.001; collision mesh filename=../../sensors/vt_refine_tactile/r1_pro_gripper_finger_link2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; visual mesh filename=../../sensors/vt_refine_tactile/r1_pro_gripper_finger_link2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
- added link right_gripper_tactile_pad1, mass 0.001; collision mesh filename=../../sensors/vt_refine_tactile/r1_pro_gripper_finger_link1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; visual mesh filename=../../sensors/vt_refine_tactile/r1_pro_gripper_finger_link1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
- added link right_gripper_tactile_pad2, mass 0.001; collision mesh filename=../../sensors/vt_refine_tactile/r1_pro_gripper_finger_link2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; visual mesh filename=../../sensors/vt_refine_tactile/r1_pro_gripper_finger_link2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
Joints:
- added joint left_gripper_tactile_pad1_joint: type fixed, parent left_gripper_finger_link1, child left_gripper_tactile_pad1, origin xyz=0 0 0 rpy=0 0 0, axis 0 0 0
- added joint left_gripper_tactile_pad2_joint: type fixed, parent left_gripper_finger_link2, child left_gripper_tactile_pad2, origin xyz=0 0 0 rpy=0 0 0, axis 0 0 0
- added joint right_gripper_tactile_pad1_joint: type fixed, parent right_gripper_finger_link1, child right_gripper_tactile_pad1, origin xyz=0 0 0 rpy=0 0 0, axis 0 0 0
- added joint right_gripper_tactile_pad2_joint: type fixed, parent right_gripper_finger_link2, child right_gripper_tactile_pad2, origin xyz=0 0 0 rpy=0 0 0, axis 0 0 0

Commit message: Remove tactile sensors.

File: source/assembly_benchmark/assembly_benchmark/assets/robots/r1_pro/robot.urdf (robot description, URDF)
Before this commit: robot r1_pro_with_gripper, 40 links, 39 joints
Links:
- removed link left_gripper_tactile_pad1
- removed link left_gripper_tactile_pad2
- removed link right_gripper_tactile_pad1
- removed link right_gripper_tactile_pad2
Joints:
- removed joint left_gripper_tactile_pad1_joint
- removed joint left_gripper_tactile_pad2_joint
- removed joint right_gripper_tactile_pad1_joint
- removed joint right_gripper_tactile_pad2_joint
