Commit message: Update Piper arm velocity limit from 5 m/s to 3 m/s.

File: source/assembly_benchmark/assembly_benchmark/assets/robots/piper/piper_description.urdf (robot description, URDF)
Before this commit: robot piper, 8 links, 7 joints
Joints:
- joint joint1: limit lower=-2.6179938 upper=2.6179938 effort=100 velocity=5 -> lower=-2.6179938 upper=2.6179938 effort=100 velocity=3
- joint joint2: limit lower=0 upper=3.1415926 effort=100 velocity=5 -> lower=0 upper=3.1415926 effort=100 velocity=3
- joint joint3: limit lower=-2.9670597 upper=0 effort=100 velocity=5 -> lower=-2.9670597 upper=0 effort=100 velocity=3
- joint joint4: limit lower=-1.7453292 upper=1.7453292 effort=100 velocity=5 -> lower=-1.7453292 upper=1.7453292 effort=100 velocity=3
- joint joint5: limit lower=-1.2217304 upper=1.2217304 effort=100 velocity=5 -> lower=-1.2217304 upper=1.2217304 effort=100 velocity=3
- joint joint6: limit lower=-2.0943951 upper=2.0943951 effort=100 velocity=5 -> lower=-2.0943951 upper=2.0943951 effort=100 velocity=3
